File: ECAD/BRAIN_BOARD.kicad_pcb (KiCad board)
At the start: 4 copper layers, 99.5 x 92.2 mm, 131 parts, among them J1 VH, J10 PH-3, J11 MTA-4, J12 JST_EH-14, J13 CRASH, J2 USB4105-GF-A (USB-C), J3 ZH-3, J4 MTA-5, J5 TC2030-NL, J6 HOME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

Commit message: Added stitching vias
Parts:
- moved C47 0.09 mm to (61.7, 146.8)
Routing:
- net +3.3V: track 134.6 -> 118.6 mm
- net GND: track 161.1 -> 161.2 mm, vias 120 -> 245
- added copper zone on B.Cu, net GND
